File: hardware/electronic/PowerSupply.sch (KiCad schematic (older format))
At the start: 21 parts, among them J8 Battery Connector, Q3 TSM850N06CX, U10 MIC5504-3.3YM5, U2 LMV321, U3 74LVC1G14, U4 MAX40200, U5 74LVC2G02, U6 MCP3421A0T-ECH, U7 MCP73831-2-OT

Commit message: Rescued schematic symbols since LMRHAT.lib didn't get saved
Parts:
- Q3: symbol LMRHAT:TSM850N06CX -> LMRHAT-rescue:TSM850N06CX-LMRHAT
- U4: symbol LMRHAT:MAX40200 -> LMRHAT-rescue:MAX40200-LMRHAT
Changed lines of the file:
@@
 $EndComp
 $Comp
-L LMRHAT:GND #PWR?
+L LMRHAT-rescue:GND-LMRHAT #PWR?
 U 1 1 5C105974
 P 9600 4400
@@
 $EndComp
 $Comp
-L LMRHAT:GND #PWR?
+L LMRHAT-rescue:GND-LMRHAT #PWR?
 U 1 1 5C10597A
 P 8500 3950
@@
 $EndComp
 $Comp
-L LMRHAT:GND #PWR?
+L LMRHAT-rescue:GND-LMRHAT #PWR?
 U 1 1 5C105985
 P 8000 3850
@@
 	9400 5550 9400 5450
 $Comp
-L LMRHAT:GND #PWR?
+L LMRHAT-rescue:GND-LMRHAT #PWR?
 U 1 1 5C10599F
 P 8900 6050
@@
 $EndComp
 $Comp
-L LMRHAT:GND #PWR?
+L LMRHAT-rescue:GND-LMRHAT #PWR?
 U 1 1 5C1059A5
 P 8400 6050
@@
 $EndComp
 $Comp
-L LMRHAT:GND #PWR?
+L LMRHAT-rescue:GND-LMRHAT #PWR?
 U 1 1 5C1059C9
 P 7400 5550
@@
 	7400 5500 7400 5550
 $Comp
-L LMRHAT:+Vopt #PWR?
+L LMRHAT-rescue:+Vopt-LMRHAT #PWR?
 U 1 1 5C1059E8
 P 1800 5100
@@
 	9400 5150 9400 3800
 $Comp
-L LMRHAT:MAX40200 U?
+L LMRHAT-rescue:MAX40200-LMRHAT U?
 U 1 1 5C1058DD
 P 3700 5250
@@
 	2300 6300 2200 6300
 $Comp
-L LMRHAT:GND #PWR?
+L LMRHAT-rescue:GND-LMRHAT #PWR?
 U 1 1 5C0622C2
 P 2600 6400
@@
 	2600 6300 2500 6300
 $Comp
-L LMRHAT:GND #PWR?
+L LMRHAT-rescue:GND-LMRHAT #PWR?
 U 1 1 5C0693A3
 P 2200 7100
@@
 	1800 5200 1800 6600
 $Comp
-L LMRHAT:+Vhandoff #PWR0124
+L LMRHAT-rescue:+Vhandoff-LMRHAT #PWR0124
 U 1 1 5C0889E9
 P 2200 5950
@@
 	4250 5200 4000 5200
 $Comp
-L LMRHAT:GND #PWR?
+L LMRHAT-rescue:GND-LMRHAT #PWR?
 U 1 1 5C0DDED0
 P 4100 5500
@@
 	1400 2300 1800 2300
 $Comp
-L LMRHAT:GND #PWR?
+L LMRHAT-rescue:GND-LMRHAT #PWR?
 U 1 1 5C1140D4
 P 2100 2800
@@
 $EndComp
 $Comp
-L LMRHAT:GND #PWR?
+L LMRHAT-rescue:GND-LMRHAT #PWR?
 U 1 1 5C12CE12
 P 9400 6050
@@
 Connection ~ 1800 2300
 $Comp
-L LMRHAT:GND #PWR?
+L LMRHAT-rescue:GND-LMRHAT #PWR?
 U 1 1 5C18B7A9
 P 1600 2000
@@
 CHARGE_EN
 $Comp
-L LMRHAT:+Vopt #PWR?
+L LMRHAT-rescue:+Vopt-LMRHAT #PWR?
 U 1 1 5C1B8268
 P 6700 3100
@@
 PWR_EN
 $Comp
-L LMRHAT:TSM850N06CX Q3
+L LMRHAT-rescue:TSM850N06CX-LMRHAT Q3
 U 1 1 5C1CC748
 P 2550 5300
@@
 	2900 4000 2900 5200
 $Comp
-L LMRHAT:GND #PWR?
+L LMRHAT-rescue:GND-LMRHAT #PWR?
 U 1 1 5C1EA973
 P 2500 4300
@@
 	2500 4300 2500 4200
 $Comp
-L LMRHAT:+Vhandoff #PWR0149
+L LMRHAT-rescue:+Vhandoff-LMRHAT #PWR0149
 U 1 1 5C1ED985
 P 1900 3600
@@
 $EndComp
 $Comp
-L LMRHAT:+Vhandoff #PWR0150
+L LMRHAT-rescue:+Vhandoff-LMRHAT #PWR0150
 U 1 1 5C1F7656
 P 5000 1700
@@
 $EndComp
 $Comp
-L LMRHAT:+Vhandoff #PWR0151
+L LMRHAT-rescue:+Vhandoff-LMRHAT #PWR0151
 U 1 1 5C1F776D
 P 5500 1700
@@
 $EndComp
 $Comp
-L LMRHAT:GND #PWR?
+L LMRHAT-rescue:GND-LMRHAT #PWR?
 U 1 1 5C1F77D8
 P 5000 2100
@@
 $EndComp
 $Comp
-L LMRHAT:GND #PWR?
+L LMRHAT-rescue:GND-LMRHAT #PWR?
 U 1 1 5C1F7961
 P 5500 2100
@@
 Note:\nCHARGE_EN is HIGH when Vopt exceeds BATT+. This signals\nthat the Pi is being powered by an external source, so the\nbattery should be disconnected and the charger enabled.
 $Comp
-L LMRHAT:+Vhandoff #PWR0139
+L LMRHAT-rescue:+Vhandoff-LMRHAT #PWR0139
 U 1 1 5C20F628
 P 1500 2800
@@
 Connection ~ 1800 2400
 $Comp
-L LMRHAT:+Vhandoff #PWR0147
+L LMRHAT-rescue:+Vhandoff-LMRHAT #PWR0147
 U 1 1 5C23087A
 P 4200 2000
@@
 	4200 2250 4200 2000
 $Comp
-L LMRHAT:+Vhandoff #PWR0148
+L LMRHAT-rescue:+Vhandoff-LMRHAT #PWR0148
 U 1 1 5C23A73B
 P 3500 1850
@@
 	9600 3900 9600 4400
 $Comp
-L LMRHAT:+3.3V #PWR0145
+L LMRHAT-rescue:+3.3V-LMRHAT #PWR0145
 U 1 1 5C044873
 P 9200 2850

Commit message: Updated layout and schematic to match board dimensions of 50x80mm
Parts:
- added TP10, TP11, TP5, TP6, TP7, TP8, TP9: (no value), TestPoint:TestPoint_Pad_D1.0mm, symbol Connector:TestPoint
Connections:
- net +handoff: now also TP5.1
- net BATT_CHARGE: now also TP10.1
- net CHARGE_EN: now also TP7.1
- net PWR_STATUS: now also TP8.1
- net SW_PWR: now also TP9.1
- net at Q3.2 (D), U10.1 (VIN), U10.3 (EN)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: now also TP6.1
- net at R19.2, R20.1, U6.1 (Vin+): now also TP11.1
Changed lines of the file:
@@
 U 1 1 5C1CC748
 P 2550 5300
+AR Path="/5C1CC748" Ref="Q3"  Part="1"
+AR Path="/5C0F7799/5C1CC748" Ref="Q3"  Part="1"
 F 0 "Q3" V 2893 5300 50  0000 C CNN
 F 1 "TSM850N06CX" V 2802 5300 50  0000 C CNN
@@
 Connection ~ 2900 4000
 Wire Wire Line
-	2900 4000 2900 5200
+	2900 4000 2900 4600
 $Comp
 L LMRHAT-rescue:GND-LMRHAT #PWR?
@@
 U 1 1 5C044873
 P 9200 2850
+AR Path="/5C044873" Ref="#PWR0145"  Part="1"
+AR Path="/5C0F7799/5C044873" Ref="#PWR0145"  Part="1"
 F 0 "#PWR0145" H 9200 2700 50  0001 C CNN
 F 1 "+3.3V" H 9215 3023 50  0000 C CNN
@@
 	1    0    0    -1
 $EndComp
+Text GLabel 5450 4250 0    39   Input ~ 0
+CHARGE_EN
+Text GLabel 5450 4350 0    50   Input ~ 0
+PWR_STATUS
+Text GLabel 5450 4450 0    50   Input ~ 0
+SW_PWR
+$Comp
+L Connector:TestPoint TP11
+U 1 1 5C576412
+P 9600 5550
+F 0 "TP11" V 9554 5738 50  0000 L CNN
+F 1 " " V 9645 5738 50  0000 L CNN
+F 2 "TestPoint:TestPoint_Pad_D1.0mm" H 9800 5550 50  0001 C CNN
+F 3 "~" H 9800 5550 50  0001 C CNN
+	1    9600 5550
+	0    1    1    0
+$EndComp
+Wire Wire Line
+	9600 5550 9400 5550
+Text GLabel 5450 4550 0    50   Input ~ 0
+BATT_CHARGE
+$Comp
+L Connector:TestPoint TP6
+U 1 1 5C578C68
+P 2900 4600
+F 0 "TP6" V 2854 4788 50  0000 L CNN
+F 1 " " V 2945 4788 50  0000 L CNN
+F 2 "TestPoint:TestPoint_Pad_D1.0mm" H 3100 4600 50  0001 C CNN
+F 3 "~" H 3100 4600 50  0001 C CNN
+	1    2900 4600
+	0    1    1    0
+$EndComp
+Connection ~ 2900 4600
+Wire Wire Line
+	2900 4600 2900 5200
+$Comp
+L Connector:TestPoint TP5
+U 1 1 5C578E00
+P 1900 3800
+F 0 "TP5" V 2000 3950 50  0000 C CNN
+F 1 " " V 2004 3874 50  0000 C CNN
+F 2 "TestPoint:TestPoint_Pad_D1.0mm" H 2100 3800 50  0001 C CNN
+F 3 "~" H 2100 3800 50  0001 C CNN
+	1    1900 3800
+	0    -1   -1   0
+$EndComp
+Connection ~ 1900 3800
+$Comp
+L Connector:TestPoint TP7
+U 1 1 5C57919C
+P 5550 4250
+F 0 "TP7" V 5504 4438 50  0000 L CNN
+F 1 " " V 5595 4438 50  0000 L CNN
+F 2 "TestPoint:TestPoint_Pad_D1.0mm" H 5750 4250 50  0001 C CNN
+F 3 "~" H 5750 4250 50  0001 C CNN
+	1    5550 4250
+	0    1    1    0
+$EndComp
+$Comp
+L Connector:TestPoint TP8
+U 1 1 5C579272
+P 5550 4350
+F 0 "TP8" V 5504 4538 50  0000 L CNN
+F 1 " " V 5595 4538 50  0000 L CNN
+F 2 "TestPoint:TestPoint_Pad_D1.0mm" H 5750 4350 50  0001 C CNN
+F 3 "~" H 5750 4350 50  0001 C CNN
+	1    5550 4350
+	0    1    1    0
+$EndComp
+$Comp
+L Connector:TestPoint TP9
+U 1 1 5C5792C0
+P 5550 4450
+F 0 "TP9" V 5504 4638 50  0000 L CNN
+F 1 " " V 5595 4638 50  0000 L CNN
+F 2 "TestPoint:TestPoint_Pad_D1.0mm" H 5750 4450 50  0001 C CNN
+F 3 "~" H 5750 4450 50  0001 C CNN
+	1    5550 4450
+	0    1    1    0
+$EndComp
+$Comp
+L Connector:TestPoint TP10
+U 1 1 5C579308
+P 5550 4550
+F 0 "TP10" V 5504 4738 50  0000 L CNN
+F 1 " " V 5595 4738 50  0000 L CNN
+F 2 "TestPoint:TestPoint_Pad_D1.0mm" H 5750 4550 50  0001 C CNN
+F 3 "~" H 5750 4550 50  0001 C CNN
+	1    5550 4550
+	0    1    1    0
+$EndComp
+Wire Wire Line
+	5550 4550 5450 4550
+Wire Wire Line
+	5450 4450 5550 4450
+Wire Wire Line
+	5550 4350 5450 4350
+Wire Wire Line
+	5450 4250 5550 4250
 $EndSCHEMATC
